File: MiCS_Sensor/MiCS_Sensor.kicad_pcb (KiCad board)
At the start: 2 copper layers, 22 x 26 mm, 17 parts, among them J1 Conn_01x04, J2 Conn_01x04, J3 Conn_01x04, Q1 2N7002, U1 MICS-4514, U2 TLC2272

Commit message: update version
Connections:
- R2 pad 1: /PRE_HEALTING -> /IO1
- U2 pad 1: /ADC_OX -> /AIN
- U2 pad 2: /ADC_OX -> /AIN
Routing:
- net /IO1: track 0.00 -> 32.4 mm, vias 0 -> 1
- net /AIN: track 0.00 -> 16.1 mm, vias 0 -> 1
- net /ADC_OX: track 1.27 -> 0.00 mm
- net GND: vias 4 -> 9
