File: MiCS_Sensor/MiCS_Sensor.kicad_sch (KiCad schematic)
At the start: 15 parts, among them J1 Conn_01x04, J2 Conn_01x04, J3 Conn_01x04, Q1 2N7002, U1 MICS-4514, U2 TLC2272

Commit message: update version
Parts:
- C1: value 0.1uF -> 10uF
Connections:
- net ADC_OX is gone; now on net AIN: U2.1, U2.2 (-)
- net PRE_HEALTING is gone; now on net IO1: R2.1
Changed lines of the file:
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@@
-    (effects (font (size 1.27 1.27)) (justify left bottom))
-  )
-  (label "ADC_OX" (at 134.747 106.7816 0)
     (effects (font (size 1.27 1.27)) (justify left bottom))
   )
@@
     (effects (font (size 1.27 1.27)) (justify left bottom))
   )
+  (label "AIN" (at 134.747 106.7816 0)
+    (effects (font (size 1.27 1.27)) (justify left bottom))
+  )
   (label "SDA" (at 236.1438 108.9914 0)
     (effects (font (size 1.27 1.27)) (justify left bottom))
@@
   (label "SCL" (at 236.1438 106.4514 0)
     (effects (font (size 1.27 1.27)) (justify left bottom))
-  )
-  (label "PRE_HEALTING" (at 85.725 81.3816 270)
-    (effects (font (size 1.27 1.27)) (justify right bottom))
   )
   (label "CO2" (at 152.019 103.7336 180)
@@
   (label "RX" (at 235.585 82.677 0)
     (effects (font (size 1.27 1.27)) (justify left bottom))
+  )
+  (label "IO1" (at 85.725 81.3816 180)
+    (effects (font (size 1.27 1.27)) (justify right bottom))
   )
   (label "AIN" (at 234.95 69.1896 0)
@@
       (effects (font (size 1.27 1.27)) hide)
     )
-    (property "Datasheet" "~" (id 3) (at 195.0466 68.1736 0)
+    (property "Datasheet" "08055C104M4T4A" (id 3) (at 195.0466 68.1736 0)
       (effects (font (size 1.27 1.27)) hide)
     )
@@
       (effects (font (size 1.27 1.27)) (justify left))
     )
-    (property "Value" "0.1uF" (id 1) (at 210.4644 69.3165 0)
+    (property "Value" "10uF" (id 1) (at 210.4644 69.3165 0)
       (effects (font (size 1.27 1.27)) (justify left))
     )
@@
       (effects (font (size 1.27 1.27)) hide)
     )
-    (property "Datasheet" "~" (id 3) (at 207.391 68.0466 0)
+    (property "Datasheet" "08055C104M4T4A" (id 3) (at 207.391 68.0466 0)
       (effects (font (size 1.27 1.27)) hide)
     )
@@
     )
     (path "/7aa5b753-3f12-4da1-96d4-171b87ce771f"
-      (reference "C1") (unit 1) (value "0.1uF") (footprint "Capacitor_SMD:C_0805_2012Metric")
+      (reference "C1") (unit 1) (value "10uF") (footprint "Capacitor_SMD:C_0805_2012Metric")
     )
     (path "/184cca5c-19ba-4bd7-8ba4-09a50fb0236b"

Commit message: update notes on schematic
Other:
- note added: "133 ohms"
- note added: "16.58 mA"
- note added: "20.24 mA"
- note added: "Q1 On - 0.6072v Q1 Off - 0.4974v"
- note added: "Q1 On - 12.29mW Q1 Off - 8.25mW"
- note added: "Q1 On - 2.69v Q1 Off - 2.20v"
Changed lines of the file:
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@@
     (stroke (width 0) (type default) (color 0 0 0 0))
+  )
+  (text "20.24 mA" (at 102.616 75.946 0)
+    (effects (font (size 1.27 1.27)) (justify left bottom))
+  )
+  (text "Q1 On - 0.6072v \nQ1 Off - 0.4974v " (at 97.028 72.644 0)
+    (effects (font (size 1.27 1.27)) (justify left bottom))
+  )
+  (text "Q1 On - 2.69v \nQ1 Off - 2.20v " (at 157.1498 58.9026 180)
+    (effects (font (size 1.27 1.27)) (justify right bottom))
+  )
+  (text "Q1 On - 12.29mW \nQ1 Off - 8.25mW " (at 97.028 68.58 0)
+    (effects (font (size 1.27 1.27)) (justify left bottom))
+  )
+  (text "133 ohms" (at 145.7198 62.1284 0)
+    (effects (font (size 1.27 1.27)) (justify left bottom))
+  )
+  (text "16.58 mA" (at 115.316 89.408 90)
+    (effects (font (size 1.27 1.27)) (justify left bottom))
   )
   (label "NO2" (at 125.095 68.4276 180)
@@
       (effects (font (size 1.27 1.27)) hide)
     )
+    (pin "1")
+    (pin "2")
+    (pin "3")
     (pin "5")
     (pin "6")
     (pin "7")
+    (pin "4")
+    (pin "8")
   )
   (symbol (lib_id "citizen_sensor-rescue:MICS-4514-electroniccats-citizen_sensor-rescue") (at 162.941 70.9676 0) (unit 1)
@@
   (symbol (lib_id "Amplifier_Operational:OPA1602") (at 123.825 106.7816 0) (unit 3)
     (in_bom yes) (on_board yes)
-    (property "Reference" "U2" (id 0) (at 122.7582 105.6132 0)
-      (effects (font (size 1.27 1.27)) (justify left))
-    )
-    (property "Value" "TLC2272" (id 1) (at 122.7582 107.9246 0)
+    (property "Reference" "U2" (id 0) (at 121.8184 107.061 0)
+      (effects (font (size 1.27 1.27)) (justify left))
+    )
+    (property "Value" "TLC2272" (id 1) (at 122.7582 112.3188 0)
       (effects (font (size 1.27 1.27)) (justify left))
     )
@@
       (effects (font (size 1.27 1.27)) hide)
     )
+    (pin "1")
+    (pin "2")
+    (pin "3")
+    (pin "5")
+    (pin "6")
+    (pin "7")
     (pin "4")
     (pin "8")
@@
       (effects (font (size 1.27 1.27)) (justify left))
     )
-    (property "Value" "2N7002" (id 1) (at 97.79 77.0636 0)
+    (property "Value" "2N7002" (id 1) (at 109.728 89.662 90)
       (effects (font (size 1.27 1.27)) (justify left))
     )
@@
     (pin "2")
     (pin "3")
+    (pin "5")
+    (pin "6")
+    (pin "7")
+    (pin "4")
+    (pin "8")
   )
   (symbol (lib_id "Connector_Generic:Conn_01x04") (at 244.3734 103.9114 0) (unit 1)
